Commit message: added collision parameters to urdf

File: urdf/hubert.urdf (robot description, URDF)
Before this commit: robot hubert, 5 links, 4 joints
Links:
- link base_link: geometry collision box size=0.055 0.02 0.02; visual box size=0.055 0.02 0.02
- link robot_arm: geometry collision box size=0.088 0.02 0.02; visual box size=0.088 0.02 0.02
- link robot_body: geometry collision box size=0.315 0.02 0.02; visual box size=0.315 0.02 0.02
- link robot_elbow: geometry collision box size=0.204 0.02 0.02; visual box size=0.204 0.02 0.02
- link robot_shoulder: geometry collision box size=0.216 0.02 0.02; visual box size=0.216 0.02 0.02
Joints:
- joint elbow_joint: limit lower=-1.57 upper=0.0 effort=1000.0 velocity=0.5 -> lower=-0.785 upper=0.785 effort=1000.0 velocity=0.5
- joint shoulder_joint: limit lower=-1.57 upper=0 effort=1000.0 velocity=0.5 -> lower=-0.785 upper=0.785 effort=1000.0 velocity=0.5
