Commit message: created new package and update move_ee

File: src/move_ee/move_ee/urdf/hubert.urdf (robot description, URDF)
Before this commit: robot hubert, 5 links, 4 joints
Joints:
- joint base_joint: limit lower=-1.57 upper=1.57 effort=1000.0 velocity=0.5 -> lower=0 upper=3.14 effort=1000.0 velocity=0.5
- joint elbow_joint: limit lower=-0.785 upper=0.785 effort=1000.0 velocity=0.5 -> lower=-0 upper=1.57075 effort=1000.0 velocity=0.5
- joint shoulder_joint: limit lower=-0.785 upper=0.785 effort=1000.0 velocity=0.5 -> lower=0 upper=3.14 effort=1000.0 velocity=0.5
