Commit message: changes for ee link and joint

File: src/hubert_grp/urdf/hubert.urdf (robot description, URDF)
Before this commit: robot hubert, 5 links, 4 joints
Links:
- added link end_effector; collision box size=0.15 0.02 0.02; visual box size=0.204 0.02 0.02
Joints:
- added joint end_effector_joint: type fixed, parent robot_elbow, child end_effector, origin xyz=0.015 -0.15 -0.005 rpy= 0 0 0, axis 0 0 1

Commit message: made changes for rviz control to work

File: src/hubert_grp/urdf/hubert.urdf (robot description, URDF)
Before this commit: robot hubert, 6 links, 5 joints
Links:
- link end_effector: geometry collision box size=0.05 0.02 0.02; visual box size=0.05 0.02 0.02

Commit message: updated visual component

File: src/hubert_grp/urdf/hubert.urdf (robot description, URDF)
Before this commit: robot hubert, 6 links, 5 joints
Joints:
- joint end_effector_joint: axis 0 0 1 -> (none)
